Commit message: finalize the simulation

File: autonomous_turret/models/turret/turret.urdf (robot description, URDF)
Before this commit: robot two_joint_robot, 6 links, 5 joints
Links:
- added link base_footprint
- link base_link: mass 1 -> 10
- link ir_sensor: geometry collision box size=0.01 0.01 0.01; visual box size=0.01 0.01 0.01
- link led_link: geometry collision sphere radius=0.01; visual sphere radius=0.01
Joints:
- added joint base_footprint_joint: type fixed, parent base_footprint, child base_link, origin xyz=0 0 0 rpy=0 0 0

Commit message: add sound

File: autonomous_turret/models/turret/turret.urdf (robot description, URDF)
Before this commit: robot two_joint_robot, 7 links, 6 joints
Links:
- removed link led_link
- removed link rotator_2
- link ir_sensor: geometry collision box size=0.05 0.05 0.05; visual box size=0.05 0.05 0.05
- link rotator_1: geometry collision cylinder length=0.2 radius=0.1; visual cylinder length=0.2 radius=0.1
- link turret_endpoint: geometry collision cylinder length=0.2 radius=0.03; visual cylinder length=0.2 radius=0.03
Joints:
- removed joint led_joint
- removed joint rotator_2_joint
- joint ir_sensor_joint: origin xyz=0 0.02 0 rpy=0 0 0 -> xyz=0 0.1 0.18 rpy=-1.57 0 0; parent turret_endpoint -> rotator_1
- joint turret_endpoint_joint: origin xyz=0 0 0 rpy=1.57 0 0 -> xyz=0 0.2 0.15 rpy=1.57 0 0; parent rotator_2 -> rotator_1

Commit message: add image

File: autonomous_turret/models/turret/turret.urdf (robot description, URDF)
Before this commit: robot two_joint_robot, 7 links, 6 joints
Links:
- removed link ir_sensor
- removed link led_link
- removed link rotator_2
- added link camera_sensor; collision box size=0.01 0.01 0.01; visual box size=0.05 0.05 0.05
- link rotator_1: geometry collision cylinder length=0.1 radius=0.1; visual cylinder length=0.1 radius=0.1
- link turret_endpoint: geometry collision box size=0.02 0.02 0.2; visual box size=0.02 0.02 0.2
Joints:
- removed joint led_joint
- removed joint rotator_2_joint
- joint ir_sensor_joint: child ir_sensor -> camera_sensor; origin xyz=0 0.02 0 rpy=0 0 0 -> xyz=0 0. 0.15 rpy=0 0 -1.57; parent turret_endpoint -> rotator_1
- joint turret_endpoint_joint: parent rotator_2 -> rotator_1
